Commit message: feat: train with imitation

File: src/ainex_description/urdf/ainex.urdf (robot description, URDF)
Before this commit: robot ainex, 28 links, 27 joints
Links:
- link l_ank_roll_link: geometry collision box size=0.12 0.08 0.004; visual mesh filename=package://ainex_description/meshes/l_ank_roll_link.STL
- link r_ank_roll_link: geometry collision box size=0.12 0.08 0.004; visual mesh filename=package://ainex_description/meshes/r_ank_roll_link.STL
